Commit message: Update somewhat working go1 model
Previous error was joint limits set from [-360,-360]. Corrected to [-360,360] and some other minor changes
Current problems:
- Try publishing a stand command but leg lifts upwards

File: quad_simulator/go1_description/urdf/go1.urdf (robot description, URDF)
Before this commit: robot go1_description, 38 links, 37 joints
Joints:
- joint 0: origin xyz=0 0.08 0 rpy=0 0 0 -> xyz=0 0.08 0 rpy=0 1.57079632679 0
- joint 1: limit lower=-6.28318530718 upper=-6.28318530718 effort=23.7 velocity=30.1 -> lower=-6.28318530718 upper=6.28318530718 effort=23.7 velocity=30.1; origin xyz=0 0 -0.213 rpy=0 0 0 -> xyz=0 0 -0.213 rpy=0 -3.14159265359 0
- joint 2: origin xyz=0 0.08 0 rpy=0 0 0 -> xyz=0 0.08 0 rpy=0 1.57079632679 0
- joint 3: limit lower=-6.28318530718 upper=-6.28318530718 effort=23.7 velocity=30.1 -> lower=-6.28318530718 upper=6.28318530718 effort=23.7 velocity=30.1; origin xyz=0 0 -0.213 rpy=0 0 0 -> xyz=0 0 -0.213 rpy=0 -3.14159265359 0
- joint 4: origin xyz=0 -0.08 0 rpy=0 0 0 -> xyz=0 -0.08 0 rpy=0 1.57079632679 0
- joint 5: limit lower=-6.28318530718 upper=-6.28318530718 effort=23.7 velocity=30.1 -> lower=-6.28318530718 upper=6.28318530718 effort=23.7 velocity=30.1; origin xyz=0 0 -0.213 rpy=0 0 0 -> xyz=0 0 -0.213 rpy=0 -3.14159265359 0
- joint 6: origin xyz=0 -0.08 0 rpy=0 0 0 -> xyz=0 -0.08 0 rpy=0 1.57079632679 0
- joint 7: limit lower=-6.28318530718 upper=-6.28318530718 effort=23.7 velocity=30.1 -> lower=-6.28318530718 upper=6.28318530718 effort=23.7 velocity=30.1; origin xyz=0 0 -0.213 rpy=0 0 0 -> xyz=0 0 -0.213 rpy=0 -3.14159265359 0

File: quad_simulator/go1_description/xacro/const.xacro (robot description, xacro)
@@ -35,9 +35,9 @@
     <xacro:property name="hip_velocity_max" value="30.1"/>
     <xacro:property name="hip_torque_max" value="23.7"/>
-    <xacro:property name="thigh_max" value="170"/>
-    <xacro:property name="thigh_min" value="-38"/>
+    <xacro:property name="thigh_max" value="170"/> <!-- Original: 170 -->
+    <xacro:property name="thigh_min" value="-38"/> <!-- Original: -38 -->
     <xacro:property name="thigh_velocity_max" value="30.1"/>
     <xacro:property name="thigh_torque_max" value="23.7"/>
-    <xacro:property name="calf_max" value="-360"/> <!-- Original: -48 -->
+    <xacro:property name="calf_max" value="360"/> <!-- Original: -48 -->
     <xacro:property name="calf_min" value="-360"/> <!-- Original: -156 --> <!-- Question: Initial Orientation: -180 (-pi) so pass min... -->
     <xacro:property name="calf_velocity_max" value="30.1"/>

File: quad_simulator/go1_description/xacro/gazebo.xacro (robot description, xacro)
@@ -3,11 +3,11 @@
     <!-- ros_control plugin -->
     <gazebo>
-        <!--<plugin name="gazebo_ros_control" filename="libgazebo_ros_control.so">
-            <robotNamespace>/go1</robotNamespace>
+        <plugin name="gazebo_ros_control" filename="libgazebo_ros_control.so">
+            <robotNamespace>/robot_1</robotNamespace>
             <robotSimType>gazebo_ros_control/DefaultRobotHWSim</robotSimType>
-        </plugin>-->
-        <!-- <plugin filename="libground_truth_estimator.so" name="ground_truth_estimator">
+        </plugin>
+        <plugin filename="libground_truth_estimator.so" name="ground_truth_estimator">
             <updateRateHZ>500.0</updateRateHZ>
-        </plugin> -->
+        </plugin>
     </gazebo>
     <!-- Show the trajectory of trunk center. -->
@@ -207,4 +207,5 @@
         </sensor>
     </gazebo> -->
+    <!-- Bumper plugin for contact sensors -->
     <!-- Make a macro for this later (low priority) -->
     <gazebo reference="toe0">
@@ -294,5 +295,5 @@
     </gazebo> -->
     <gazebo reference="body">
-        <material>Gazebo/Grey</material>
+        <material>Gazebo/White</material>
         <turnGravityOff>false</turnGravityOff>
     </gazebo>

File: quad_simulator/go1_description/xacro/leg.xacro (robot description, xacro)
@@ -100,5 +100,5 @@
         <joint name="${hipJointName}" type="revolute">
             <!-- <origin rpy="0 ${PI/2} 0" xyz="0 ${thigh_offset*mirror} 0"/> -->
-            <origin rpy="0 0 0" xyz="0 ${thigh_offset*mirror} 0"/>
+            <origin rpy="0 ${PI/2} 0" xyz="0 ${thigh_offset*mirror} 0"/>
             <parent link="hip${suffix}"/>
             <child link="upper${suffix}"/>
@@ -117,5 +117,5 @@
             </visual>
             <collision name="lower${suffix}_collision">
-                <origin rpy="0 ${PI/2.0} 0" xyz="0 0 ${-calf_length/2.0}"/>
+                <origin rpy="0 ${PI/2.0} 0" xyz="0 0 ${-calf_length/2.0}"/> <!-- origin rpy="0 ${PI/2.0} 0" xyz="0 0 ${-calf_length/2.0}"/ -->
                 <geometry>
                     <box size="${calf_length} ${calf_width} ${calf_height}"/>
@@ -124,5 +124,5 @@
             <inertial>
                 <origin rpy="0 0 0" xyz="${calf_com_x} ${calf_com_y} ${calf_com_z}"/>
-                <mass value="${calf_mass}"/>
+                <mass value="${calf_mass}"/> <!-- ${calf_mass} -->
                 <inertia
                     ixx="${calf_ixx}" ixy="${calf_ixy}" ixz="${calf_ixz}"
@@ -134,5 +134,5 @@
         <joint name="${kneeJointName}" type="revolute">
             <!-- <origin rpy="0 ${-PI} 0" xyz="0 0 ${-thigh_length}"/> -->
-            <origin rpy="0 0 0" xyz="0 0 ${-thigh_length}"/>
+            <origin rpy="0 ${-PI} 0" xyz="0 0 ${-thigh_length}"/>
             <parent link="upper${suffix}"/>
             <child link="lower${suffix}"/>

Commit message: Working go1 model with quad-sdk
Small bug fixes to create a working model of go1 that is able to load, stand, and execute plan properly
- Changed sitting initial angle as original angle caused meshes within one another causing tricky bugs
- Incorporated go1 into local_planner (Specified if robot_name==go1, load a1 system_id, etc.
- Update urdf and xacro files to working one (previous commits may not have been updated)

File: quad_simulator/go1_description/urdf/go1.urdf (robot description, URDF)
Before this commit: robot go1_description, 38 links, 37 joints
Joints:
- joint 0: axis 0 1 0 -> 0 -1 0; limit lower=-0.663225115758 upper=2.96705972839 effort=23.7 velocity=30.1 -> lower=-6.28318530718 upper=6.28318530718 effort=23.7 velocity=30.1
- joint 1: origin xyz=0 0 -0.213 rpy=0 -3.14159265359 0 -> xyz=0 0 -0.213 rpy=0 -3.05008995494 0
- joint 2: axis 0 1 0 -> 0 -1 0; limit lower=-0.663225115758 upper=2.96705972839 effort=23.7 velocity=30.1 -> lower=-6.28318530718 upper=6.28318530718 effort=23.7 velocity=30.1
- joint 3: origin xyz=0 0 -0.213 rpy=0 -3.14159265359 0 -> xyz=0 0 -0.213 rpy=0 -3.05008995494 0
- joint 4: axis 0 1 0 -> 0 -1 0; limit lower=-0.663225115758 upper=2.96705972839 effort=23.7 velocity=30.1 -> lower=-6.28318530718 upper=6.28318530718 effort=23.7 velocity=30.1
- joint 5: origin xyz=0 0 -0.213 rpy=0 -3.14159265359 0 -> xyz=0 0 -0.213 rpy=0 -3.05008995494 0
- joint 6: axis 0 1 0 -> 0 -1 0; limit lower=-0.663225115758 upper=2.96705972839 effort=23.7 velocity=30.1 -> lower=-6.28318530718 upper=6.28318530718 effort=23.7 velocity=30.1
- joint 7: origin xyz=0 0 -0.213 rpy=0 -3.14159265359 0 -> xyz=0 0 -0.213 rpy=0 -3.05008995494 0

File: quad_simulator/go1_description/xacro/const.xacro (robot description, xacro)
@@ -29,18 +29,18 @@
     <xacro:property name="hip_offset" value="0.08"/>
     <!-- joint limits -->
-    <xacro:property name="damping" value="0.01"/>
-    <xacro:property name="friction" value="0.2"/>
+    <xacro:property name="damping" value="0.01"/> <!-- Original value: 0.01 -->
+    <xacro:property name="friction" value="0.2"/> <!-- Original value: 0.2 -->
     <xacro:property name="hip_max" value="60"/>
     <xacro:property name="hip_min" value="-60"/>
-    <xacro:property name="hip_velocity_max" value="30.1"/>
-    <xacro:property name="hip_torque_max" value="23.7"/>
-    <xacro:property name="thigh_max" value="170"/> <!-- Original: 170 -->
-    <xacro:property name="thigh_min" value="-38"/> <!-- Original: -38 -->
-    <xacro:property name="thigh_velocity_max" value="30.1"/>
-    <xacro:property name="thigh_torque_max" value="23.7"/>
+    <xacro:property name="hip_velocity_max" value="30.1"/> <!-- Original value: 30.1 -->
+    <xacro:property name="hip_torque_max" value="23.7"/> <!-- Original value: 23.7 -->
+    <xacro:property name="thigh_max" value="360"/> <!-- Original: 170 -->
+    <xacro:property name="thigh_min" value="-360"/> <!-- Original: -38 -->
+    <xacro:property name="thigh_velocity_max" value="30.1"/> <!-- Original value: 30.1 -->
+    <xacro:property name="thigh_torque_max" value="23.7"/> <!-- Original value: 23.7 -->
     <xacro:property name="calf_max" value="360"/> <!-- Original: -48 -->
     <xacro:property name="calf_min" value="-360"/> <!-- Original: -156 --> <!-- Question: Initial Orientation: -180 (-pi) so pass min... -->
-    <xacro:property name="calf_velocity_max" value="30.1"/>
-    <xacro:property name="calf_torque_max" value="23.7"/>
+    <xacro:property name="calf_velocity_max" value="30.1"/> <!-- Original value: 30.1 -->
+    <xacro:property name="calf_torque_max" value="23.7"/> <!-- Original value: 23.7 -->
     <!-- dynamics inertial value        total 12.84kg -->
     <!-- trunk -->

File: quad_simulator/go1_description/xacro/gazebo.xacro (robot description, xacro)
@@ -4,5 +4,4 @@
     <gazebo>
         <plugin name="gazebo_ros_control" filename="libgazebo_ros_control.so">
-            <robotNamespace>/robot_1</robotNamespace>
             <robotSimType>gazebo_ros_control/DefaultRobotHWSim</robotSimType>
         </plugin>

File: quad_simulator/go1_description/xacro/leg.xacro (robot description, xacro)
@@ -103,5 +103,5 @@
             <parent link="hip${suffix}"/>
             <child link="upper${suffix}"/>
-            <axis xyz="0 1 0"/>
+            <axis xyz="0 -1 0"/>
             <dynamics damping="${damping}" friction="${friction}"/>
             <limit effort="${thigh_torque_max}" velocity="${thigh_velocity_max}" lower="${thigh_min*PI/180.0}" upper="${thigh_max*PI/180.0}"/>
@@ -134,5 +134,5 @@
         <joint name="${kneeJointName}" type="revolute">
             <!-- <origin rpy="0 ${-PI} 0" xyz="0 0 ${-thigh_length}"/> -->
-            <origin rpy="0 ${-PI} 0" xyz="0 0 ${-thigh_length}"/>
+            <origin rpy="0 ${-PI/1.03} 0" xyz="0 0 ${-thigh_length}"/>
             <parent link="upper${suffix}"/>
             <child link="lower${suffix}"/>

File: quad_simulator/go1_description/xacro/robot.xacro (robot description, xacro)
@@ -112,22 +112,22 @@
     </link>
     <!-- Legs Xacro -->
-    <!-- FL -->
+    <!--FL-->
     <xacro:leg suffix="0" mirror="1" mirror_dae="True" front_hind="1" front_hind_dae="True"
-                hipJointName="0" kneeJointName="1" abductionJointName="8">
+               hipJointName="0" kneeJointName="1" abductionJointName="8">
         <origin rpy="0 0 0" xyz="${leg_offset_x} ${leg_offset_y} 0"/>
     </xacro:leg>
-    <!-- RL -->
+    <!--RL-->
     <xacro:leg suffix="1" mirror="1" mirror_dae="True" front_hind="-1" front_hind_dae="False"
-                hipJointName="2" kneeJointName="3" abductionJointName="9">
+               hipJointName="2" kneeJointName="3" abductionJointName="9">
         <origin rpy="0 0 0" xyz="${-leg_offset_x} ${leg_offset_y} 0"/>
     </xacro:leg>
-    <!-- FR -->
+    <!--FR-->
     <xacro:leg suffix="2" mirror="-1" mirror_dae="False" front_hind="1" front_hind_dae="True"
-                hipJointName="4" kneeJointName="5" abductionJointName="10">
+               hipJointName="4" kneeJointName="5" abductionJointName="10">
         <origin rpy="0 0 0" xyz="${leg_offset_x} ${-leg_offset_y} 0"/>
     </xacro:leg>
-    <!-- RR -->
+    <!--RR-->
     <xacro:leg suffix="3" mirror="-1" mirror_dae="False" front_hind="-1" front_hind_dae="False"
-                hipJointName="6" kneeJointName="7" abductionJointName="11">
+               hipJointName="6" kneeJointName="7" abductionJointName="11">
         <origin rpy="0 0 0" xyz="${-leg_offset_x} ${-leg_offset_y} 0"/>
     </xacro:leg>

Commit message: Updated go1 model
Disabled self-collision:
- Disabled self collision to have initial stand position at 0 0.76 1.52
- Lower leg origin at 0 -PI 0

File: quad_simulator/go1_description/urdf/go1.urdf (robot description, URDF)
Before this commit: robot go1_description, 38 links, 37 joints
Joints:
- joint 1: origin xyz=0 0 -0.213 rpy=0 -3.05008995494 0 -> xyz=0 0 -0.213 rpy=0 -3.14159265359 0
- joint 3: origin xyz=0 0 -0.213 rpy=0 -3.05008995494 0 -> xyz=0 0 -0.213 rpy=0 -3.14159265359 0
- joint 5: origin xyz=0 0 -0.213 rpy=0 -3.05008995494 0 -> xyz=0 0 -0.213 rpy=0 -3.14159265359 0
- joint 7: origin xyz=0 0 -0.213 rpy=0 -3.05008995494 0 -> xyz=0 0 -0.213 rpy=0 -3.14159265359 0

File: quad_simulator/go1_description/xacro/gazebo.xacro (robot description, xacro)
@@ -322,5 +322,5 @@
         <mu1>0.2</mu1>
         <mu2>0.2</mu2>
-        <self_collide>1</self_collide>
+        <self_collide>0</self_collide>
         <material>Gazebo/DarkGrey</material>
         <kp  value="1000000.0"/>
@@ -330,10 +330,10 @@
         <mu1>0.2</mu1>
         <mu2>0.2</mu2>
-        <self_collide>1</self_collide>
+        <self_collide>0</self_collide>
     </gazebo>
     <gazebo reference="toe0">
         <mu1>0.6</mu1>
         <mu2>0.6</mu2>
-        <self_collide>1</self_collide>
+        <self_collide>0</self_collide>
         <material>Gazebo/DarkGrey</material>
         <kp  value="1000000.0"/>
@@ -349,5 +349,5 @@
         <mu1>0.2</mu1>
         <mu2>0.2</mu2>
-        <self_collide>1</self_collide>
+        <self_collide>0</self_collide>
         <material>Gazebo/DarkGrey</material>
         <kp  value="1000000.0"/>
@@ -357,10 +357,10 @@
         <mu1>0.2</mu1>
         <mu2>0.2</mu2>
-        <self_collide>1</self_collide>
+        <self_collide>0</self_collide>
     </gazebo>
     <gazebo reference="toe1">
         <mu1>0.6</mu1>
         <mu2>0.6</mu2>
-        <self_collide>1</self_collide>
+        <self_collide>0</self_collide>
         <material>Gazebo/DarkGrey</material>
         <kp  value="1000000.0"/>
@@ -376,5 +376,5 @@
         <mu1>0.2</mu1>
         <mu2>0.2</mu2>
-        <self_collide>1</self_collide>
+        <self_collide>0</self_collide>
         <material>Gazebo/DarkGrey</material>
         <kp  value="1000000.0"/>
@@ -384,10 +384,10 @@
         <mu1>0.2</mu1>
         <mu2>0.2</mu2>
-        <self_collide>1</self_collide>
+        <self_collide>0</self_collide>
     </gazebo>
     <gazebo reference="toe2">
         <mu1>0.6</mu1>
         <mu2>0.6</mu2>
-        <self_collide>1</self_collide>
+        <self_collide>0</self_collide>
         <material>Gazebo/DarkGrey</material>
         <kp  value="1000000.0"/>
@@ -403,5 +403,5 @@
         <mu1>0.2</mu1>
         <mu2>0.2</mu2>
-        <self_collide>1</self_collide>
+        <self_collide>0</self_collide>
         <material>Gazebo/DarkGrey</material>
         <kp  value="1000000.0"/>
@@ -411,10 +411,10 @@
         <mu1>0.2</mu1>
         <mu2>0.2</mu2>
-        <self_collide>1</self_collide>
+        <self_collide>0</self_collide>
     </gazebo>
     <gazebo reference="toe3">
         <mu1>0.6</mu1>
         <mu2>0.6</mu2>
-        <self_collide>1</self_collide>
+        <self_collide>0</self_collide>
         <material>Gazebo/DarkGrey</material>
         <kp  value="1000000.0"/>

File: quad_simulator/go1_description/xacro/leg.xacro (robot description, xacro)
@@ -134,5 +134,5 @@
         <joint name="${kneeJointName}" type="revolute">
             <!-- <origin rpy="0 ${-PI} 0" xyz="0 0 ${-thigh_length}"/> -->
-            <origin rpy="0 ${-PI/1.03} 0" xyz="0 0 ${-thigh_length}"/>
+            <origin rpy="0 ${-PI} 0" xyz="0 0 ${-thigh_length}"/>
             <parent link="upper${suffix}"/>
             <child link="lower${suffix}"/>
