Commit message: Major overhaul for Cpp Google Style Code

File: quad_simulator/a1_description/xacro/leg.xacro (robot description, xacro)
@@ -88,5 +88,5 @@
         </link>
         <joint name="${hipJointName}" type="revolute">
-            <origin rpy="0 ${PI/2.0} 0" xyz="0 ${thigh_offset*mirror} 0"/>
+            <origin rpy="0 ${PI/2.0} 0" xyz="0 ${thigh_offset*mirror} 0"/> <!-- <origin rpy="0 ${PI/2.0} 0" xyz="0 ${thigh_offset*mirror} 0"/> -->
             <parent link="hip${suffix}"/>
             <child link="upper${suffix}"/>
@@ -116,5 +116,5 @@
         </link>
         <joint name="${kneeJointName}" type="revolute">
-            <origin rpy="0 ${-PI} 0" xyz="0 0 ${-thigh_length}"/>
+            <origin rpy="0 ${-PI} 0" xyz="0 0 ${-thigh_length}"/> <!-- <origin rpy="0 ${-PI} 0" xyz="0 0 ${-thigh_length}"/> -->
             <parent link="upper${suffix}"/>
             <child link="lower${suffix}"/>
