Commit message: Large number of changes
This update change consists generally of the following... Modified URDF model s.t. for Gazebo-9, inertia problems for root link is not a problem (may cause issues with some of how quad-sdk reads the linkages). Change starting positions s.t. step_10cm_local_min spawns w/o dropping into infinite pit. Lastly, made lots of comments in GBPL, local planner, etc. to help myself in reading the code and keeping up with the intricate data flow.

File: quad_simulator/spirit_description/urdf/spirit.urdf (robot description, URDF)
Before this commit: robot spirit, 19 links, 18 joints
Links:
- added link base
Joints:
- added joint base_body_joint: type fixed, parent base, child body

Commit message: URDF & SDF Implementation Trial Run
Consists of 2 updates:
- Commenting control plugin code
- Attempt to convert spirit.urdf -> spirit.sdf (Failed)... Some discrepancies from urdf and sdf files that I assume are manual changes
TODO: Attempt to use urdf and xacro files from main branch and work from there

File: quad_simulator/spirit_description/urdf/spirit.urdf (robot description, URDF)
Before this commit: robot spirit, 17 links, 16 joints
Links:
- added link body_inertia, mass 7.388
- link body: mass 7.388 -> None
Joints:
- added joint body_body_inertia: type fixed, parent body, child body_inertia

File: quad_simulator/spirit_description/urdf/spirit_gazebo.urdf.xacro (robot description, xacro)
@@ -26,68 +26,78 @@
 	<!-- bodyLength + hipdx should be equal to front to back hip distance -->
 	<!-- dy +  dPodAxisToEdge + upperLegWidth should be equal to the center to toe distance along y axis-->
-	<xacro:property name="pi" value="3.14159265359"/>
-	<xacro:property name="bodyLength" value="0.335"/>
-	<xacro:property name="bodyWidth" value="0.24"/>
-	<xacro:property name="bodyHeight" value="0.104"/>
-	<xacro:property name="bodyMass" value="5.75"/>
-	<xacro:property name="podMass" value="0.575"/>
-	<xacro:property name="upperLegMass" value="0.775"/>
-	<xacro:property name="upperLegIxx" value="0.00005"/> <!-- guess -->
-	<xacro:property name="upperLegIyy" value="0.001"/> <!-- guess -->
-	<xacro:property name="upperLegIzz" value="0.001"/> <!-- guess -->
-	<xacro:property name="lowerLegMass" value="0.075"/>
-	<xacro:property name="lowerLegIxx" value="0.000005"/> <!-- guess -->
-	<xacro:property name="lowerLegIyy" value="0.0001"/> <!-- guess -->
-	<xacro:property name="lowerLegIzz" value="0.0001"/> <!-- guess -->
-	<xacro:property name="toeMass" value="0.015"/>
-	<xacro:property name="upperLegLength" value="0.206"/>
-	<xacro:property name="upperLegWidth" value="0.022"/>
-	<xacro:property name="upperLegHeight" value="0.055"/>
-	<xacro:property name="lowerLegLength" value="0.206"/>
-	<xacro:property name="lowerLegRadius" value="0.013"/> <!--visual only-->
-	<xacro:property name="podLength" value="0.08"/>
-	<xacro:property name="podRadius" value="0.055"/>
-	<xacro:property name="dPodAxisToEdge" value="0.028"/> <!--center of pod cylinder to the ab axis-->
-	<xacro:property name="abOffs" value="0.10098"/>
-	<xacro:property name="dx" value="0.2263"/>
-	<xacro:property name="dy" value="0.07"/>
-	<xacro:property name="toeRadius" value="0.02"/>
-	<xacro:property name="toeOffset" value="0.0"/>
-	<xacro:property name="toeStiffness" value="30000.0"/>
-	<xacro:property name="toeDamping" value="1000.0"/>
-	<xacro:property name="toeSpinningFriction" value="0.3"/>
-	<xacro:property name="toeFriction" value="100.0"/>
-	<xacro:property name="toeLateralFriction" value="50.0"/>
-	<xacro:property name="abKinLimit" value="0.707"/>
-	<xacro:property name="abSpeedLimit" value="30"/>
-	<xacro:property name="abEffortLimit" value="40"/>
-	<xacro:property name="jointSpeedLimit" value="30"/>
-	<xacro:property name="jointEffortLimit" value="40"/>
+	<xacro:property name="pi" value="3.14159265359" />
+	<xacro:property name="bodyLength" value="0.335" />
+	<xacro:property name="bodyWidth" value="0.24" />
+	<xacro:property name="bodyHeight" value="0.104" />
+	<xacro:property name="bodyMass" value="5.75" />
+	<xacro:property name="podMass" value="0.575" />
+	<xacro:property name="upperLegMass" value="0.775" />
+	<xacro:property name="upperLegIxx" value="0.00005" /> <!-- guess -->
+	<xacro:property name="upperLegIyy" value="0.001" /> <!-- guess -->
+	<xacro:property name="upperLegIzz" value="0.001" /> <!-- guess -->
+	<xacro:property name="lowerLegMass" value="0.075" />
+	<xacro:property name="lowerLegIxx" value="0.000005" /> <!-- guess -->
+	<xacro:property name="lowerLegIyy" value="0.0001" /> <!-- guess -->
+	<xacro:property name="lowerLegIzz" value="0.0001" /> <!-- guess -->
+	<xacro:property name="toeMass" value="0.015" />
+	<xacro:property name="upperLegLength" value="0.206" />
+	<xacro:property name="upperLegWidth" value="0.022" />
+	<xacro:property name="upperLegHeight" value="0.055" />
+	<xacro:property name="lowerLegLength" value="0.206" />
+	<xacro:property name="lowerLegRadius" value="0.013" /> <!--visual only-->
+	<xacro:property name="podLength" value="0.08" />
+	<xacro:property name="podRadius" value="0.055" />
+	<xacro:property name="dPodAxisToEdge" value="0.028" /> <!--center of pod cylinder to the ab axis-->
+	<xacro:property name="abOffs" value="0.10098" />
+	<xacro:property name="dx" value="0.2263" />
+	<xacro:property name="dy" value="0.07" />
+	<xacro:property name="toeRadius" value="0.02" />
+	<xacro:property name="toeOffset" value="0.0" />
+	<xacro:property name="toeStiffness" value="30000.0" />
+	<xacro:property name="toeDamping" value="1000.0" />
+	<xacro:property name="toeSpinningFriction" value="0.3" />
+	<xacro:property name="toeFriction" value="100.0" />
+	<xacro:property name="toeLateralFriction" value="50.0" />
+	<xacro:property name="abKinLimit" value="0.707" />
+	<xacro:property name="abSpeedLimit" value="30" />
+	<xacro:property name="abEffortLimit" value="40" />
+	<xacro:property name="jointSpeedLimit" value="30" />
+	<xacro:property name="jointEffortLimit" value="40" />
+	<!--link name="body_dummy">
+		<inertial>
+			<mass value="${bodyMass}" />
+			<inertia ixx="0.05" ixy="0" ixz="0" iyy="0.1" iyz="0" izz="0.1" />
+		</inertial>
+	</link>
+	<joint name="dummy_joint" type="fixed">
+		<parent link="body_dummy" />
+		<child link="body" />
+	</joint-->
 	<!-- Body -->
 	<link name="body">
 		<visual>
-			<origin rpy="0 0 0" xyz="0 0 0"/>
+			<origin rpy="0 0 0" xyz="0 0 0" />
 			<geometry>
-				<box size="${bodyLength} ${bodyWidth} ${bodyHeight}"/>
+				<box size="${bodyLength} ${bodyWidth} ${bodyHeight}" />
 			</geometry>
-			<material name="darkgray"/>
+			<material name="darkgray" />
 		</visual>
 		<inertial>
-			<mass value="${bodyMass}"/>
+			<mass value="${bodyMass}" />
 			<!-- Uniform box -->
 			<!-- <inertia ixx="1/12*${bodyMass}*(${bodyWidth}*${bodyWidth} + ${bodyHeight}*${bodyHeight})"  ixy="0"  ixz="0" iyy="1/12*${bodyMass}*(${bodyLength}*${bodyLength} + ${bodyHeight}*${bodyHeight})" iyz="0" izz="1/12*${bodyMass}*(${bodyLength}*${bodyLength} + ${bodyWidth}*${bodyWidth})"/> -->
-			<inertia ixx="0.05"  ixy="0"  ixz="0" iyy="0.1" iyz="0" izz="0.1" />
+			<inertia ixx="0.05" ixy="0" ixz="0" iyy="0.1" iyz="0" izz="0.1" />
 		</inertial>
 		<!-- Just copy geometry for collision -->
 		<collision>
-		<origin rpy="0 0 0" xyz="0 0 0"/>
+			<origin rpy="0 0 0" xyz="0 0 0" />
 			<geometry>
-				<box size="${bodyLength} ${bodyWidth} ${bodyHeight}"/>
+				<box size="${bodyLength} ${bodyWidth} ${bodyHeight}" />
 			</geometry>
 		</collision>
 	</link>
 	<gazebo reference="body">
-    	<material>Gazebo/Black</material>
-  	</gazebo>
+		<material>Gazebo/Black</material>
+	</gazebo>
 	<!-- Define our leg macro -->
 	<xacro:macro name="leg" params="suffix left front hipJointName kneeJointName abductionJointName hipJointLowerLimit hipJointUpperLimit color">
@@ -95,161 +105,161 @@
 		<link name="hip${suffix}">
 			<visual>
-				<origin rpy="${pi/2} 0 0" xyz="${front * 0} ${left * (dPodAxisToEdge)} 0"/>
-				<geometry>
-					<cylinder length="${podLength}" radius="${podRadius}"/>
+				<origin rpy="${pi/2} 0 0" xyz="${front * 0} ${left * (dPodAxisToEdge)} 0" />
+				<geometry>
+					<cylinder length="${podLength}" radius="${podRadius}" />
 				</geometry>
 			</visual>
 			<collision>
-				<origin rpy="${pi/2} 0 0" xyz="0 ${left * (dPodAxisToEdge)} 0"/>
-				<geometry>
-					<cylinder length="${podLength}" radius="${podRadius}"/>
+				<origin rpy="${pi/2} 0 0" xyz="0 ${left * (dPodAxisToEdge)} 0" />
+				<geometry>
+					<cylinder length="${podLength}" radius="${podRadius}" />
 				</geometry>
 			</collision>
 			<inertial>
-				<mass value="${podMass}"/>
+				<mass value="${podMass}" />
 				<!-- <inertia ixx="1/12*${podMass}*${podLength}*${podLength} + 1/4*${podMass}*${podRadius}*${podRadius}"  ixy="0"  ixz="0" iyy="1/12*${podMass}*${podLength}*${podLength} + 1/4*${podMass}*${podRadius}*${podRadius}" iyz="0" izz="1/2*${podMass}*${podRadius}*$
 				{podRadius}" /> -->
-				<inertia ixx="0.00066963541"  ixy="0"  ixz="0" iyy="0.00066963541" iyz="0" izz="0.0008696875" />
+				<inertia ixx="0.00066963541" ixy="0" ixz="0" iyy="0.00066963541" iyz="0" izz="0.0008696875" />
 			</inertial>
 		</link>
 		<gazebo reference="hip${suffix}">
 			<material>Gazebo/Grey</material>
-  		</gazebo>
+		</gazebo>
 		<!-- Abduction joint. Joint names are: 8 9 10 11 -->
 		<joint name="${abductionJointName}" type="revolute">
-			<parent link="body"/>
-			<child link="hip${suffix}"/>
-			<axis xyz="1 0 0"/>
-			<origin xyz="${front * dx} ${left * dy} 0"/>
-			<limit effort="${abEffortLimit}" velocity="${abSpeedLimit}" lower="${-abKinLimit}" upper="${abKinLimit}"/>
-			<dynamics damping="0.0" friction="0.0"/>
+			<parent link="body" />
+			<child link="hip${suffix}" />
+			<axis xyz="1 0 0" />
+			<origin xyz="${front * dx} ${left * dy} 0" />
+			<limit effort="${abEffortLimit}" velocity="${abSpeedLimit}" lower="${-abKinLimit}" upper="${abKinLimit}" />
+			<dynamics damping="0.0" friction="0.0" />
 		</joint>
 		<!-- Transmission elements required for Gazebo -->
 		<transmission name="transmission_${abductionJointName}">
-    		<type>transmission_interface/SimpleTransmission</type>
-    		<joint name="${abductionJointName}">
-      			<hardwareInterface>hardware_interface/EffortJointInterface</hardwareInterface>
-    		</joint>
-    		<actuator name="motor_${abductionJointName}">
-      			<hardwareInterface>EffortJointInterface</hardwareInterface>
-      			<mechanicalReduction>1</mechanicalReduction>
-    		</actuator>
-  		</transmission>
+			<type>transmission_interface/SimpleTransmission</type>
+			<joint name="${abductionJointName}">
+				<hardwareInterface>hardware_interface/EffortJointInterface</hardwareInterface>
+			</joint>
+			<actuator name="motor_${abductionJointName}">
+				<hardwareInterface>EffortJointInterface</hardwareInterface>
+				<mechanicalReduction>1</mechanicalReduction>
+			</actuator>
+		</transmission>
 		<!-- Upper leg -->
 		<link name="upper${suffix}">
 			<visual>
-				<origin rpy="0 0 0" xyz="-${upperLegLength/2} ${-left*upperLegWidth} 0"/>
-				<geometry>
-					<box size="${upperLegLength} ${upperLegWidth} ${upperLegHeight}"/>
-				</geometry>
-				<material name="silver"/>
+				<origin rpy="0 0 0" xyz="-${upperLegLength/2} ${-left*upperLegWidth} 0" />
+				<geometry>
+					<box size="${upperLegLength} ${upperLegWidth} ${upperLegHeight}" />
+				</geometry>
+				<material name="silver" />
 			</visual>
 			<collision>
-				<origin rpy="0 0 0" xyz="-${upperLegLength/2} ${-left*upperLegWidth} 0"/>
-				<geometry>
-					<box size="${upperLegLength} ${upperLegWidth} ${upperLegHeight}"/>
+				<origin rpy="0 0 0" xyz="-${upperLegLength/2} ${-left*upperLegWidth} 0" />
+				<geometry>
+					<box size="${upperLegLength} ${upperLegWidth} ${upperLegHeight}" />
 				</geometry>
 			</collision>
 			<inertial>
-				<mass value="${upperLegMass}"/>
-				<inertia ixx="${upperLegIxx}"  ixy="0" ixz="0" iyy="${upperLegIyy}" iyz="0" izz="${upperLegIzz}"/>
+				<mass value="${upperLegMass}" />
+				<inertia ixx="${upperLegIxx}" ixy="0" ixz="0" iyy="${upperLegIyy}" iyz="0" izz="${upperLegIzz}" />
 			</inertial>
 		</link>
 		<gazebo reference="upper${suffix}">
 			<material>Gazebo/DarkGrey</material>
-  		</gazebo>
+		</gazebo>
 		<!-- Hip joint. (Motor to upper leg). Joint names are: 0 2 4 6 -->
 		<joint name="${hipJointName}" type="revolute">
-			<parent link="hip${suffix}"/>
-			<child link="upper${suffix}"/>
-			<axis xyz="0 -1 0"/>
-			<origin xyz="${front * 0} ${left * abOffs} 0"/> <!--  rpy="0 -0.3 0" -->
-			<limit effort="${jointEffortLimit}" velocity="${jointSpeedLimit}" lower="${hipJointLowerLimit}" upper="${hipJointUpperLimit}"/>
-			<dynamics damping="0.0" friction="0.0"/>
+			<parent link="hip${suffix}" />
+			<child link="upper${suffix}" />
+			<axis xyz="0 -1 0" />
+			<origin xyz="${front * 0} ${left * abOffs} 0" /> <!--  rpy="0 -0.3 0" -->
+			<limit effort="${jointEffortLimit}" velocity="${jointSpeedLimit}" lower="${hipJointLowerLimit}" upper="${hipJointUpperLimit}" />
+			<dynamics damping="0.0" friction="0.0" />
 		</joint>
 		<!-- Transmission elements required for Gazebo -->
 		<transmission name="transmission_${hipJointName}">
-    		<type>transmission_interface/SimpleTransmission</type>
-    		<joint name="${hipJointName}">
-      			<hardwareInterface>hardware_interface/EffortJointInterface</hardwareInterface>
-    		</joint>
-    		<actuator name="motor_${hipJointName}">
-      			<hardwareInterface>EffortJointInterface</hardwareInterface>
-      			<mechanicalReduction>1</mechanicalReduction>
-    		</actuator>
-  		</transmission>
+			<type>transmission_interface/SimpleTransmission</type>
+			<joint name="${hipJointName}">
+				<hardwareInterface>hardware_interface/EffortJointInterface</hardwareInterface>
+			</joint>
+			<actuator name="motor_${hipJointName}">
+				<hardwareInterface>EffortJointInterface</hardwareInterface>
+				<mechanicalReduction>1</mechanicalReduction>
+			</actuator>
+		</transmission>
 		<!-- Lower leg -->
 		<link name="lower${suffix}">
 			<visual>
-				<origin rpy="0 ${pi/2} 0" xyz="${lowerLegLength/2} 0 0"/>
-				<geometry>
-					<cylinder length="${lowerLegLength}" radius="${lowerLegRadius}"/>
-				</geometry>
-				<material name="darkgray"/>
+				<origin rpy="0 ${pi/2} 0" xyz="${lowerLegLength/2} 0 0" />
+				<geometry>
+					<cylinder length="${lowerLegLength}" radius="${lowerLegRadius}" />
+				</geometry>
+				<material name="darkgray" />
 			</visual>
 			<collision>
-				<origin rpy="0 ${pi/2} 0" xyz="${lowerLegLength/2} 0 0"/>
-				<geometry>
-					<cylinder length="${lowerLegLength}" radius="${lowerLegRadius}"/>
+				<origin rpy="0 ${pi/2} 0" xyz="${lowerLegLength/2} 0 0" />
+				<geometry>
+					<cylinder length="${lowerLegLength}" radius="${lowerLegRadius}" />
 				</geometry>
 			</collision>
 			<inertial>
-				<mass value="${lowerLegMass}"/>
-				<inertia ixx="${lowerLegIxx}"  ixy="0" ixz="0" iyy="${lowerLegIyy}" iyz="0" izz="${lowerLegIzz}"/>
+				<mass value="${lowerLegMass}" />
+				<inertia ixx="${lowerLegIxx}" ixy="0" ixz="0" iyy="${lowerLegIyy}" iyz="0" izz="${lowerLegIzz}" />
 			</inertial>
 		</link>
 		<gazebo reference="lower${suffix}">
 			<material>Gazebo/Grey</material>
-  		</gazebo>
+		</gazebo>
 		<!-- Knee joint. Joint names are: 1 3 5 7 -->
 		<joint name="${kneeJointName}" type="revolute">
-			<parent link="upper${suffix}"/>
-			<child link="lower${suffix}"/>
-			<axis xyz="0 1 0"/>
-			<origin xyz="-${upperLegLength} 0 0"/> <!--rpy="0 0.5 0"-->
-			<limit effort="${jointEffortLimit}" velocity="${jointSpeedLimit}" lower="0" upper="${pi}"/>
-			<dynamics damping="0.0" friction="0.0"/>
+			<parent link="upper${suffix}" />
+			<child link="lower${suffix}" />
+			<axis xyz="0 1 0" />
+			<origin xyz="-${upperLegLength} 0 0" /> <!--rpy="0 0.5 0"-->
+			<limit effort="${jointEffortLimit}" velocity="${jointSpeedLimit}" lower="0" upper="${pi}" />
+			<dynamics damping="0.0" friction="0.0" />
 		</joint>
 		<!-- Transmission elements required for Gazebo -->
 		<transmission name="transmission_${kneeJointName}">
-    		<type>transmission_interface/SimpleTransmission</type>
-    		<joint name="${kneeJointName}">
-      			<hardwareInterface>hardware_interface/EffortJointInterface</hardwareInterface>
-    		</joint>
-    		<actuator name="motor_${kneeJointName}">
-      			<hardwareInterface>EffortJointInterface</hardwareInterface>
-      			<mechanicalReduction>1</mechanicalReduction>
-    		</actuator>
-  		</transmission>
+			<type>transmission_interface/SimpleTransmission</type>
+			<joint name="${kneeJointName}">
+				<hardwareInterface>hardware_interface/EffortJointInterface</hardwareInterface>
+			</joint>
+			<actuator name="motor_${kneeJointName}">
+				<hardwareInterface>EffortJointInterface</hardwareInterface>
+				<mechanicalReduction>1</mechanicalReduction>
+			</actuator>
+		</transmission>
 		<!-- Toe -->
 		<link name="toe${suffix}">
 			<contact>
-				<friction_anchor/>
-				<stiffness value="${toeStiffness}"/>
-				<damping value="${toeDamping}"/>
-				<spinning_friction value="${toeSpinningFriction}"/>
-				<lateral_friction value="${toeLateralFriction}"/>
+				<friction_anchor />
+				<stiffness value="${toeStiffness}" />
+				<damping value="${toeDamping}" />
+				<spinning_friction value="${toeSpinningFriction}" />
+				<lateral_friction value="${toeLateralFriction}" />
 			</contact>
 			<visual>
-				<origin rpy="0 0 0" xyz="0 0 0"/>
-				<geometry>
-					<sphere radius="${toeRadius}"/>
-				</geometry>
-				<material name="darkgray"/>
+				<origin rpy="0 0 0" xyz="0 0 0" />
+				<geometry>
+					<sphere radius="${toeRadius}" />
+				</geometry>
+				<material name="darkgray" />
 			</visual>
 			<collision>
-				<origin rpy="0 0 0" xyz="0 0 0"/>
-				<geometry>
-					<sphere radius="${toeRadius}"/>
+				<origin rpy="0 0 0" xyz="0 0 0" />
+				<geometry>
+					<sphere radius="${toeRadius}" />
 				</geometry>
 			</collision>
 			<inertial>
-				<mass value="${toeMass}"/>
-				<inertia ixx="0.000025"  ixy="0"  ixz="0" iyy="0.000025" iyz="0" izz="0.000025" />
+				<mass value="${toeMass}" />
+				<inertia ixx="0.000025" ixy="0" ixz="0" iyy="0.000025" iyz="0" izz="0.000025" />
 				<!-- <inertia ixx="2/5*${toeMass}*${toeRadius}*${toeRadius}"  ixy="0"  ixz="0" iyy="2/5*${toeMass}*${toeRadius}*${toeRadius}" iyz="0" izz="2/5*${toeMass}*${toeRadius}*${toeRadius}" /> -->
 			</inertial>
 		</link>
 		<gazebo reference="toe${suffix}">
-    		<material>Gazebo/Black</material>
+			<material>Gazebo/Black</material>
 			<collision>
 				<surface>
@@ -283,22 +293,22 @@
 				</surface>
 			</collision>
-  		</gazebo>
+		</gazebo>
 		<joint name="jtoe${suffix}" type="fixed">
-			<parent link="lower${suffix}"/>
-			<child link="toe${suffix}"/>
-			<origin xyz="${lowerLegLength} 0 -${toeOffset}"/>
-			<dynamics damping="0.0" friction="0.0"/>
+			<parent link="lower${suffix}" />
+			<child link="toe${suffix}" />
+			<origin xyz="${lowerLegLength} 0 -${toeOffset}" />
+			<dynamics damping="0.0" friction="0.0" />
 		</joint>
 	</xacro:macro>
 	<!-- Our four legs -->
-	<xacro:leg suffix="0" hipJointName="0" kneeJointName="1" abductionJointName="8" front="1" left="1" hipJointLowerLimit="${-2*pi}" hipJointUpperLimit="${2*pi}" color="darkgray"/>
- 	<xacro:leg suffix="1" hipJointName="2" kneeJointName="3" abductionJointName="9" front="-1" left="1" hipJointLowerLimit="${-2*pi}" hipJointUpperLimit="${2*pi}" color="darkgray"/>
- 	<xacro:leg suffix="2" hipJointName="4" kneeJointName="5" abductionJointName="10" front="1" left="-1" hipJointLowerLimit="${-2*pi}" hipJointUpperLimit="${2*pi}" color="red"/>
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
File: quad_simulator/spirit_description/urdf/spirit_tail_2.urdf (robot description, URDF)
Before this commit: robot spirit, 21 links, 20 joints
Links:
- removed link inertia_dummy
- removed link tail_link_0
- removed link tail_link_1
- removed link tail_mass
- link body: mass 7.388 -> 5.75
- link lower0: mass 0.096 -> 0.075
- link lower1: mass 0.096 -> 0.075
- link lower2: mass 0.096 -> 0.075
- link lower3: mass 0.096 -> 0.075
- link upper0: mass 0.792 -> 0.775
- link upper1: mass 0.792 -> 0.775
- link upper2: mass 0.792 -> 0.775
- link upper3: mass 0.792 -> 0.775
Joints:
- removed joint body_inertia_dummy
- removed joint body_tail_joint_0
- removed joint body_tail_joint_1
- removed joint tail_link_mass_joint
