Commit message: Modified state estimator plugin and mass values
Following changes were
- State estimator determined if joint was fixed -> if is -> push 0 vel & pos
- Temporary change in mass values to see if inertia was a problem
TODO: Calculate correct inertia values corresponding to the mass

File: quad_simulator/spirit_description/urdf/spirit_gazebo.urdf.xacro (robot description, xacro)
@@ -64,4 +64,14 @@
 	<xacro:property name="jointSpeedLimit" value="30" />
 	<xacro:property name="jointEffortLimit" value="40" />
+	<!-- Plugins -->
+	<gazebo>
+		<plugin name="gazebo_ros_control" filename="libgazebo_ros_control.so">
+			<robotNamespace>/spirit</robotNamespace>
+			<controlPeriod>0.002</controlPeriod>
+		</plugin>
+		<plugin name="ground_truth_estimator" filename="libground_truth_estimator.so">
+			<updateRateHz>500.0</updateRateHz>
+		</plugin>
+	</gazebo>
 	<!--link name="body_dummy">
 		<inertial>
@@ -167,4 +177,5 @@
 		</link>
 		<gazebo reference="upper${suffix}">
+			<self_collide>0</self_collide>
 			<material>Gazebo/DarkGrey</material>
 		</gazebo>
@@ -191,4 +202,5 @@
 		<!-- Lower leg -->
 		<link name="lower${suffix}">
+			<self_collide>0</self_collide>
 			<visual>
 				<origin rpy="0 ${pi/2} 0" xyz="${lowerLegLength/2} 0 0" />
@@ -261,4 +273,5 @@
 		</link>
 		<gazebo reference="toe${suffix}">
+			<self_collide>0</self_collide>
 			<material>Gazebo/Black</material>
 			<collision>
@@ -304,11 +317,75 @@
 	<xacro:leg suffix="0" hipJointName="0" kneeJointName="1" abductionJointName="8" front="1" left="1" hipJointLowerLimit="${-2*pi}" hipJointUpperLimit="${2*pi}" color="darkgray" />
 	<xacro:leg suffix="1" hipJointName="2" kneeJointName="3" abductionJointName="9" front="-1" left="1" hipJointLowerLimit="${-2*pi}" hipJointUpperLimit="${2*pi}" color="darkgray" />
-	<xacro:leg suffix="2" hipJointName="4" kneeJointName="5" abductionJointName="10" front="1" left="-1" hipJointLowerLimit="${-2*pi}" hipJointUpperLimit="${2*pi}" color="red" />
+	<xacro:leg suffix="2" hipJointName="4" kneeJointName="5" abductionJointName="10" front="1" left="-1" hipJointLowerLimit="${-2*pi}" hipJointUpperLimit="${2*pi}" color="darkgray" />
 	<xacro:leg suffix="3" hipJointName="6" kneeJointName="7" abductionJointName="11" front="-1" left="-1" hipJointLowerLimit="${-2*pi}" hipJointUpperLimit="${2*pi}" color="darkgray" />
-	<!-- Add ros_control plugin -->
-	<gazebo>
-		<plugin name="gazebo_ros_control" filename="libgazebo_ros_control.so">
-			<robotNamespace>/spirit</robotNamespace>
-		</plugin>
+	<!-- Toe Plugins -->
+	<gazebo reference="toe0">
+		<sensor name="toe0_contact" type="contact">
+			<plugin filename="libgazebo_ros_bumper.so" name="toe0_plugin">
+				<alwaysOn>true</alwaysOn>
+				<updateRate>500</updateRate>
+				<bumperTopicName>gazebo/toe0_contact_state</bumperTopicName>
+				<frameName>world</frameName>
+			</plugin>
+			<contact>
+				<collision>toe0_collision</collision>
+			</contact>
+			<update_rate>500</update_rate>
+		</sensor>
+	</gazebo>
+	<gazebo reference="toe1">
+		<sensor name="toe1_contact" type="contact">
+			<plugin filename="libgazebo_ros_bumper.so" name="toe1_plugin">
+				<alwaysOn>true</alwaysOn>
+				<updateRate>500</updateRate>
+				<bumperTopicName>gazebo/toe1_contact_state</bumperTopicName>
+				<frameName>world</frameName>
+			</plugin>
+			<contact>
+				<collision>toe1_collision</collision>
+			</contact>
+			<update_rate>500</update_rate>
+		</sensor>
+	</gazebo>
+	<gazebo reference="toe2">
+		<sensor name="toe2_contact" type="contact">
+			<plugin filename="libgazebo_ros_bumper.so" name="toe2_plugin">
+				<alwaysOn>true</alwaysOn>
+				<updateRate>500</updateRate>
+				<bumperTopicName>gazebo/toe2_contact_state</bumperTopicName>
+				<frameName>world</frameName>
+			</plugin>
+			<contact>
+				<collision>toe2_collision</collision>
+			</contact>
+			<update_rate>500</update_rate>
+		</sensor>
+	</gazebo>
+	<gazebo reference="toe3">
+		<sensor name="toe3_contact" type="contact">
+			<plugin filename="libgazebo_ros_bumper.so" name="toe3_plugin">
+				<alwaysOn>true</alwaysOn>
+				<updateRate>500</updateRate>
+				<bumperTopicName>gazebo/toe3_contact_state</bumperTopicName>
+				<frameName>world</frameName>
+			</plugin>
+			<contact>
+				<collision>toe3_collision</collision>
+			</contact>
+			<update_rate>500</update_rate>
+		</sensor>
+	</gazebo>
+	<!-- Preserve fixed joints -->
+	<gazebo reference='jtoe0'>
+		<preserveFixedJoint>true</preserveFixedJoint>
+	</gazebo>
+	<gazebo reference='jtoe1'>
+		<preserveFixedJoint>true</preserveFixedJoint>
+	</gazebo>
+	<gazebo reference='jtoe2'>
+		<preserveFixedJoint>true</preserveFixedJoint>
+	</gazebo>
+	<gazebo reference='jtoe3'>
+		<preserveFixedJoint>true</preserveFixedJoint>
 	</gazebo>
 </robot>

Commit message: Fix state estimator and urdf files for spirit

File: quad_simulator/spirit_description/urdf/spirit_gazebo.urdf.xacro (robot description, xacro)
@@ -30,10 +30,10 @@
 	<xacro:property name="bodyWidth" value="0.24" />
 	<xacro:property name="bodyHeight" value="0.104" />
-	<xacro:property name="bodyMass" value="5.75" />
+	<xacro:property name="bodyMass" value="5.75" /> <!-- Original: 5.75 -->
 	<xacro:property name="podMass" value="0.575" />
-	<xacro:property name="upperLegMass" value="0.775" />
-	<xacro:property name="upperLegIxx" value="0.00005" /> <!-- guess -->
-	<xacro:property name="upperLegIyy" value="0.001" /> <!-- guess -->
-	<xacro:property name="upperLegIzz" value="0.001" /> <!-- guess -->
+	<xacro:property name="upperLegMass" value="0.792" /> <!-- Original: 0.775 -->
+	<xacro:property name="upperLegIxx" value="0.005" /> <!-- guess --> <!-- Original: 0.005 -->
+	<xacro:property name="upperLegIyy" value="0.0070" /> <!-- guess --> <!-- Original: 0.001 -->
+	<xacro:property name="upperLegIzz" value="0.0070" /> <!-- guess --> <!-- Original: 0.0070 -->
 	<xacro:property name="lowerLegMass" value="0.075" />
 	<xacro:property name="lowerLegIxx" value="0.000005" /> <!-- guess -->
@@ -60,8 +60,8 @@
 	<xacro:property name="toeLateralFriction" value="50.0" />
 	<xacro:property name="abKinLimit" value="0.707" />
-	<xacro:property name="abSpeedLimit" value="30" />
-	<xacro:property name="abEffortLimit" value="40" />
-	<xacro:property name="jointSpeedLimit" value="30" />
-	<xacro:property name="jointEffortLimit" value="40" />
+	<xacro:property name="abSpeedLimit" value="37.7" /> <!-- Original: 37.7 -->
+	<xacro:property name="abEffortLimit" value="21" /> <!-- Original: 40 -->
+	<xacro:property name="jointSpeedLimit" value="37.7" /> <!-- Original: 30 -->
+	<xacro:property name="jointEffortLimit" value="21" /> <!-- Original: 40 -->
 	<!-- Plugins -->
 	<gazebo>
@@ -94,8 +94,8 @@
 		</visual>
 		<inertial>
-			<mass value="${bodyMass}" />
+			<mass value="7.388" /> <!--<mass value="${bodyMass}" /> -->
 			<!-- Uniform box -->
 			<!-- <inertia ixx="1/12*${bodyMass}*(${bodyWidth}*${bodyWidth} + ${bodyHeight}*${bodyHeight})"  ixy="0"  ixz="0" iyy="1/12*${bodyMass}*(${bodyLength}*${bodyLength} + ${bodyHeight}*${bodyHeight})" iyz="0" izz="1/12*${bodyMass}*(${bodyLength}*${bodyLength} + ${bodyWidth}*${bodyWidth})"/> -->
-			<inertia ixx="0.05" ixy="0" ixz="0" iyy="0.1" iyz="0" izz="0.1" />
+			<inertia ixx="0.0642434782" ixy="0" ixz="0" iyy="0.1284869565" iyz="0" izz="0.1284869565" /> <!--<inertia ixx="0.05" ixy="0" ixz="0" iyy="0.1" iyz="0" izz="0.1" />-->
 		</inertial>
 		<!-- Just copy geometry for collision -->
@@ -127,8 +127,8 @@
 			</collision>
 			<inertial>
+				<origin rpy="${pi/2} 0 0" xyz="0 ${left * (dPodAxisToEdge)} 0" />
 				<mass value="${podMass}" />
-				<!-- <inertia ixx="1/12*${podMass}*${podLength}*${podLength} + 1/4*${podMass}*${podRadius}*${podRadius}"  ixy="0"  ixz="0" iyy="1/12*${podMass}*${podLength}*${podLength} + 1/4*${podMass}*${podRadius}*${podRadius}" iyz="0" izz="1/2*${podMass}*${podRadius}*$
-				{podRadius}" /> -->
-				<inertia ixx="0.00066963541" ixy="0" ixz="0" iyy="0.00066963541" iyz="0" izz="0.0008696875" />
+				<inertia ixx="${1/12*podMass*(podLength*podLength + 3*podRadius*podRadius)}" ixy="0" ixz="0" iyy="${1/12*podMass*(podLength*podLength + 3*podRadius*podRadius)}" iyz="0" izz="${1/2*podMass*podRadius*podRadius}" /> <!-- Okay for now... forgot when cylinder is formed what direction is x pointing in -->
+				<!--inertia ixx="0.00066963541" ixy="0" ixz="0" iyy="0.00066963541" iyz="0" izz="0.0008696875" /-->
 			</inertial>
 		</link>
@@ -172,6 +172,10 @@
 			</collision>
 			<inertial>
+				<origin xyz="${-upperLegLength/2} ${-left*upperLegWidth} 0" rpy="0 0 0" />
 				<mass value="${upperLegMass}" />
-				<inertia ixx="${upperLegIxx}" ixy="0" ixz="0" iyy="${upperLegIyy}" iyz="0" izz="${upperLegIzz}" />
+				<!--<inertia ixx="${upperLegIxx}" ixy="0" ixz="0" iyy="${upperLegIyy}" iyz="0" izz="${upperLegIzz}" /> -->
+				<inertia ixx="${upperLegMass/12*(upperLegWidth*upperLegWidth + upperLegHeight*upperLegHeight)}" ixy="0" ixz="0"
+					iyy="${upperLegMass/12*(upperLegLength*upperLegLength + upperLegHeight*upperLegHeight)}" iyz="0"
+					izz="${upperLegMass/12*(upperLegWidth*upperLegWidth + upperLegLength*upperLegLength)}" />
 			</inertial>
 		</link>
@@ -217,6 +221,10 @@
 			</collision>
 			<inertial>
+				<origin xyz="${lowerLegLength/2} 0 0" rpy="0 0 0" />
 				<mass value="${lowerLegMass}" />
-				<inertia ixx="${lowerLegIxx}" ixy="0" ixz="0" iyy="${lowerLegIyy}" iyz="0" izz="${lowerLegIzz}" />
+				<!--inertia ixx="${lowerLegIxx}" ixy="0" ixz="0" iyy="${lowerLegIyy}" iyz="0" izz="${lowerLegIzz}" /-->
+				<inertia ixx="${lowerLegMass/12*(upperLegWidth*upperLegWidth + upperLegHeight*upperLegHeight)}" ixy="0" ixz="0"
+					iyy="${lowerLegMass/12*(upperLegLength*upperLegLength + upperLegHeight*upperLegHeight)}" iyz="0"
+					izz="${lowerLegMass/12*(upperLegWidth*upperLegWidth + upperLegLength*upperLegLength)}" />
 			</inertial>
 		</link>
@@ -230,5 +238,6 @@
 			<axis xyz="0 1 0" />
 			<origin xyz="-${upperLegLength} 0 0" /> <!--rpy="0 0.5 0"-->
-			<limit effort="${jointEffortLimit}" velocity="${jointSpeedLimit}" lower="0" upper="${pi}" />
+			<!--<limit effort="${jointEffortLimit}" velocity="${jointSpeedLimit}" lower="0" upper="${pi}" />-->
+			<limit effort="${32}" velocity="${25.1}" lower="-6.28" upper="${6.28}" />
 			<dynamics damping="0.0" friction="0.0" />
 		</joint>
@@ -315,8 +324,12 @@
 	</xacro:macro>
 	<!-- Our four legs -->
-	<xacro:leg suffix="0" hipJointName="0" kneeJointName="1" abductionJointName="8" front="1" left="1" hipJointLowerLimit="${-2*pi}" hipJointUpperLimit="${2*pi}" color="darkgray" />
+	<!--<xacro:leg suffix="0" hipJointName="0" kneeJointName="1" abductionJointName="8" front="1" left="1" hipJointLowerLimit="${-2*pi}" hipJointUpperLimit="${2*pi}" color="darkgray" />
 	<xacro:leg suffix="1" hipJointName="2" kneeJointName="3" abductionJointName="9" front="-1" left="1" hipJointLowerLimit="${-2*pi}" hipJointUpperLimit="${2*pi}" color="darkgray" />
 	<xacro:leg suffix="2" hipJointName="4" kneeJointName="5" abductionJointName="10" front="1" left="-1" hipJointLowerLimit="${-2*pi}" hipJointUpperLimit="${2*pi}" color="darkgray" />
-	<xacro:leg suffix="3" hipJointName="6" kneeJointName="7" abductionJointName="11" front="-1" left="-1" hipJointLowerLimit="${-2*pi}" hipJointUpperLimit="${2*pi}" color="darkgray" />
+	<xacro:leg suffix="3" hipJointName="6" kneeJointName="7" abductionJointName="11" front="-1" left="-1" hipJointLowerLimit="${-2*pi}" hipJointUpperLimit="${2*pi}" color="darkgray" />-->
+	<xacro:leg suffix="0" hipJointName="0" kneeJointName="1" abductionJointName="8" front="1" left="1" hipJointLowerLimit="${-1.57}" hipJointUpperLimit="${3.14}" color="darkgray" />
+	<xacro:leg suffix="1" hipJointName="2" kneeJointName="3" abductionJointName="9" front="-1" left="1" hipJointLowerLimit="${-1.57}" hipJointUpperLimit="${3.14}" color="darkgray" />
+	<xacro:leg suffix="2" hipJointName="4" kneeJointName="5" abductionJointName="10" front="1" left="-1" hipJointLowerLimit="${-1.57}" hipJointUpperLimit="${3.14}" color="darkgray" />
+	<xacro:leg suffix="3" hipJointName="6" kneeJointName="7" abductionJointName="11" front="-1" left="-1" hipJointLowerLimit="${-1.57}" hipJointUpperLimit="${3.14}" color="darkgray" />
 	<!-- Toe Plugins -->
 	<gazebo reference="toe0">

File: quad_simulator/spirit_description/urdf/spirit_tail_2.urdf (robot description, URDF)
Before this commit: robot spirit, 17 links, 16 joints
Links:
- link body: mass 5.75 -> 7.388
- link upper0: mass 0.775 -> 0.792
- link upper1: mass 0.775 -> 0.792
- link upper2: mass 0.775 -> 0.792
- link upper3: mass 0.775 -> 0.792
Joints:
- joint 0: limit lower=-6.28318530718 upper=6.28318530718 effort=40 velocity=30 -> lower=-1.57 upper=3.14 effort=21 velocity=37.7
- joint 1: limit lower=0 upper=3.14159265359 effort=40 velocity=30 -> lower=-6.28 upper=6.28 effort=32 velocity=25.1
- joint 10: limit lower=-0.707 upper=0.707 effort=40 velocity=30 -> lower=-0.707 upper=0.707 effort=21 velocity=37.7
- joint 11: limit lower=-0.707 upper=0.707 effort=40 velocity=30 -> lower=-0.707 upper=0.707 effort=21 velocity=37.7
- joint 2: limit lower=-6.28318530718 upper=6.28318530718 effort=40 velocity=30 -> lower=-1.57 upper=3.14 effort=21 velocity=37.7
- joint 3: limit lower=0 upper=3.14159265359 effort=40 velocity=30 -> lower=-6.28 upper=6.28 effort=32 velocity=25.1
- joint 4: limit lower=-6.28318530718 upper=6.28318530718 effort=40 velocity=30 -> lower=-1.57 upper=3.14 effort=21 velocity=37.7
- joint 5: limit lower=0 upper=3.14159265359 effort=40 velocity=30 -> lower=-6.28 upper=6.28 effort=32 velocity=25.1
- joint 6: limit lower=-6.28318530718 upper=6.28318530718 effort=40 velocity=30 -> lower=-1.57 upper=3.14 effort=21 velocity=37.7
- joint 7: limit lower=0 upper=3.14159265359 effort=40 velocity=30 -> lower=-6.28 upper=6.28 effort=32 velocity=25.1
- joint 8: limit lower=-0.707 upper=0.707 effort=40 velocity=30 -> lower=-0.707 upper=0.707 effort=21 velocity=37.7
- joint 9: limit lower=-0.707 upper=0.707 effort=40 velocity=30 -> lower=-0.707 upper=0.707 effort=21 velocity=37.7
