Commit message: Working 1-tail and 2-tail spirit model
Updates:
- Add the following spirit models: 1-tail & 2-tail model
- Update tail_controller.yaml for params of open_loop_tail
- Add tail type OPEN_LOOP in tail_type.h
- Edited controller and estimator plugin
- Add tail control config file (specific name is spirit_control_tail_dira.yaml)
- Enable open_loop parameters (e.g. switch statements, etc in controller_plugin.cpp and estimator_plugin.cpp)

File: quad_simulator/spirit_description/urdf/spirit_tail_1.urdf (robot description, URDF)
Before this commit: robot spirit, 20 links, 19 joints
Links:
- removed link tail_link_1
- link tail_link_0: geometry visual cylinder length=0.8816 radius=0.02
Joints:
- removed joint body_tail_joint_1
- joint tail_link_mass_joint: origin xyz=0 0 0.4408 -> xyz=0 0 0.8816; parent tail_link_1 -> tail_link_0
