Commit message: Modularize tail_controlller.cpp
The following are updated:
- Modularized tail_controller.cpp s.t. can have more than 2 tail option
- For tail links > 2 -> Have limp as difficult to stabilize
- Created xacro model for planar (+2 tail links) and non-planar (<= 2 tail links)
- Updated ros util to convert odom msg to eigen for > 2 tail option
- Added more models

File: quad_simulator/spirit_description/urdf/spirit_tail_10.urdf (robot description, URDF)
Before this commit: robot spirit, 19 links, 18 joints
Links:
- added link tail_link_1, mass 0.001; visual cylinder length=0.08816 radius=0.02
- added link tail_link_2, mass 0.001; visual cylinder length=0.08816 radius=0.02
- added link tail_link_3, mass 0.001; visual cylinder length=0.08816 radius=0.02
- added link tail_link_4, mass 0.001; visual cylinder length=0.08816 radius=0.02
- added link tail_link_5, mass 0.001; visual cylinder length=0.08816 radius=0.02
- added link tail_link_6, mass 0.001; visual cylinder length=0.08816 radius=0.02
- added link tail_link_7, mass 0.001; visual cylinder length=0.08816 radius=0.02
- added link tail_link_8, mass 0.001; visual cylinder length=0.08816 radius=0.02
- added link tail_link_9, mass 0.001; visual cylinder length=0.08816 radius=0.02
- link tail_link_0: geometry visual cylinder length=0.08816 radius=0.02
- link tail_mass: geometry collision sphere radius=0.04; visual sphere radius=0.04
Joints:
- added joint body_tail_joint_1: type revolute, parent tail_link_0, child tail_link_1, origin xyz=0 0 0.08816 rpy=0 0 0, axis 0 1 0, limit lower=-1.57 upper=1.57 effort=50 velocity=40
- added joint body_tail_joint_2: type revolute, parent tail_link_1, child tail_link_2, origin xyz=0 0 0.08816 rpy=0 0 0, axis 0 1 0, limit lower=-1.57 upper=1.57 effort=50 velocity=40
- added joint body_tail_joint_3: type revolute, parent tail_link_2, child tail_link_3, origin xyz=0 0 0.08816 rpy=0 0 0, axis 0 1 0, limit lower=-1.57 upper=1.57 effort=50 velocity=40
- added joint body_tail_joint_4: type revolute, parent tail_link_3, child tail_link_4, origin xyz=0 0 0.08816 rpy=0 0 0, axis 0 1 0, limit lower=-1.57 upper=1.57 effort=50 velocity=40
- added joint body_tail_joint_5: type revolute, parent tail_link_4, child tail_link_5, origin xyz=0 0 0.08816 rpy=0 0 0, axis 0 1 0, limit lower=-1.57 upper=1.57 effort=50 velocity=40
- added joint body_tail_joint_6: type revolute, parent tail_link_5, child tail_link_6, origin xyz=0 0 0.08816 rpy=0 0 0, axis 0 1 0, limit lower=-1.57 upper=1.57 effort=50 velocity=40
- added joint body_tail_joint_7: type revolute, parent tail_link_6, child tail_link_7, origin xyz=0 0 0.08816 rpy=0 0 0, axis 0 1 0, limit lower=-1.57 upper=1.57 effort=50 velocity=40
- added joint body_tail_joint_8: type revolute, parent tail_link_7, child tail_link_8, origin xyz=0 0 0.08816 rpy=0 0 0, axis 0 1 0, limit lower=-1.57 upper=1.57 effort=50 velocity=40
- added joint body_tail_joint_9: type revolute, parent tail_link_8, child tail_link_9, origin xyz=0 0 0.08816 rpy=0 0 0, axis 0 1 0, limit lower=-1.57 upper=1.57 effort=50 velocity=40
- joint body_tail_joint_0: axis 1 0 0 -> 0 1 0
- joint tail_link_mass_joint: origin xyz=0 0 0.8816 -> xyz=0 0 0.08816; parent tail_link_0 -> tail_link_9

File: quad_simulator/spirit_description/urdf/spirit_tail_2.urdf (robot description, URDF)
Before this commit: robot spirit, 20 links, 19 joints
Links:
- link tail_link_0: mass 1e-03 -> 0.001
- link tail_link_1: mass 1e-03 -> 0.001
Joints:
- joint body_tail_joint_0: limit lower=-1.57 upper=1.57 effort=50 velocity=1000000 -> lower=-1.57 upper=1.57 effort=50 velocity=40
- joint body_tail_joint_1: limit lower=-1.57 upper=1.57 effort=50 velocity=1000000 -> lower=-1.57 upper=1.57 effort=50 velocity=40

File: quad_simulator/spirit_description/urdf/spirit_tail_3.urdf (robot description, URDF)
Before this commit: robot spirit, 19 links, 18 joints
Links:
- added link tail_link_1, mass 0.001; visual cylinder length=0.293866666667 radius=0.02
- added link tail_link_2, mass 0.001; visual cylinder length=0.293866666667 radius=0.02
- link tail_link_0: geometry visual cylinder length=0.293866666667 radius=0.02
- link tail_mass: geometry collision sphere radius=0.04; visual sphere radius=0.04
Joints:
- added joint body_tail_joint_1: type revolute, parent tail_link_0, child tail_link_1, origin xyz=0 0 0.293866666667 rpy=0 0 0, axis 0 1 0, limit lower=-1.57 upper=1.57 effort=50 velocity=40
- added joint body_tail_joint_2: type revolute, parent tail_link_1, child tail_link_2, origin xyz=0 0 0.293866666667 rpy=0 0 0, axis 0 1 0, limit lower=-1.57 upper=1.57 effort=50 velocity=40
- joint body_tail_joint_0: axis 1 0 0 -> 0 1 0
- joint tail_link_mass_joint: origin xyz=0 0 0.8816 -> xyz=0 0 0.293866666667; parent tail_link_0 -> tail_link_2

File: quad_simulator/spirit_description/urdf/spirit_tail_4.urdf (robot description, URDF)
Before this commit: robot spirit, 19 links, 18 joints
Links:
- added link tail_link_1, mass 0.001; visual cylinder length=0.2204 radius=0.02
- added link tail_link_2, mass 0.001; visual cylinder length=0.2204 radius=0.02
- added link tail_link_3, mass 0.001; visual cylinder length=0.2204 radius=0.02
- link tail_link_0: geometry visual cylinder length=0.2204 radius=0.02
- link tail_mass: geometry collision sphere radius=0.04; visual sphere radius=0.04
Joints:
- added joint body_tail_joint_1: type revolute, parent tail_link_0, child tail_link_1, origin xyz=0 0 0.2204 rpy=0 0 0, axis 0 1 0, limit lower=-1.57 upper=1.57 effort=50 velocity=40
- added joint body_tail_joint_2: type revolute, parent tail_link_1, child tail_link_2, origin xyz=0 0 0.2204 rpy=0 0 0, axis 0 1 0, limit lower=-1.57 upper=1.57 effort=50 velocity=40
- added joint body_tail_joint_3: type revolute, parent tail_link_2, child tail_link_3, origin xyz=0 0 0.2204 rpy=0 0 0, axis 0 1 0, limit lower=-1.57 upper=1.57 effort=50 velocity=40
- joint body_tail_joint_0: axis 1 0 0 -> 0 1 0
- joint tail_link_mass_joint: origin xyz=0 0 0.8816 -> xyz=0 0 0.2204; parent tail_link_0 -> tail_link_3

File: quad_simulator/spirit_description/urdf/spirit_tail_5.urdf (robot description, URDF)
Before this commit: robot spirit, 19 links, 18 joints
Links:
- added link tail_link_1, mass 0.001; visual cylinder length=0.17632 radius=0.02
- added link tail_link_2, mass 0.001; visual cylinder length=0.17632 radius=0.02
- added link tail_link_3, mass 0.001; visual cylinder length=0.17632 radius=0.02
- added link tail_link_4, mass 0.001; visual cylinder length=0.17632 radius=0.02
- link tail_link_0: geometry visual cylinder length=0.17632 radius=0.02
- link tail_mass: geometry collision sphere radius=0.04; visual sphere radius=0.04
Joints:
- added joint body_tail_joint_1: type revolute, parent tail_link_0, child tail_link_1, origin xyz=0 0 0.17632 rpy=0 0 0, axis 0 1 0, limit lower=-1.57 upper=1.57 effort=50 velocity=40
- added joint body_tail_joint_2: type revolute, parent tail_link_1, child tail_link_2, origin xyz=0 0 0.17632 rpy=0 0 0, axis 0 1 0, limit lower=-1.57 upper=1.57 effort=50 velocity=40
- added joint body_tail_joint_3: type revolute, parent tail_link_2, child tail_link_3, origin xyz=0 0 0.17632 rpy=0 0 0, axis 0 1 0, limit lower=-1.57 upper=1.57 effort=50 velocity=40
- added joint body_tail_joint_4: type revolute, parent tail_link_3, child tail_link_4, origin xyz=0 0 0.17632 rpy=0 0 0, axis 0 1 0, limit lower=-1.57 upper=1.57 effort=50 velocity=40
- joint body_tail_joint_0: axis 1 0 0 -> 0 1 0
- joint tail_link_mass_joint: origin xyz=0 0 0.8816 -> xyz=0 0 0.17632; parent tail_link_0 -> tail_link_4

File: quad_simulator/spirit_description/urdf/spirit_tail_6.urdf (robot description, URDF)
Before this commit: robot spirit, 19 links, 18 joints
Links:
- added link tail_link_1, mass 0.001; visual cylinder length=0.146933333333 radius=0.02
- added link tail_link_2, mass 0.001; visual cylinder length=0.146933333333 radius=0.02
- added link tail_link_3, mass 0.001; visual cylinder length=0.146933333333 radius=0.02
- added link tail_link_4, mass 0.001; visual cylinder length=0.146933333333 radius=0.02
- added link tail_link_5, mass 0.001; visual cylinder length=0.146933333333 radius=0.02
- link tail_link_0: geometry visual cylinder length=0.146933333333 radius=0.02
- link tail_mass: geometry collision sphere radius=0.04; visual sphere radius=0.04
Joints:
- added joint body_tail_joint_1: type revolute, parent tail_link_0, child tail_link_1, origin xyz=0 0 0.146933333333 rpy=0 0 0, axis 0 1 0, limit lower=-1.57 upper=1.57 effort=50 velocity=40
- added joint body_tail_joint_2: type revolute, parent tail_link_1, child tail_link_2, origin xyz=0 0 0.146933333333 rpy=0 0 0, axis 0 1 0, limit lower=-1.57 upper=1.57 effort=50 velocity=40
- added joint body_tail_joint_3: type revolute, parent tail_link_2, child tail_link_3, origin xyz=0 0 0.146933333333 rpy=0 0 0, axis 0 1 0, limit lower=-1.57 upper=1.57 effort=50 velocity=40
- added joint body_tail_joint_4: type revolute, parent tail_link_3, child tail_link_4, origin xyz=0 0 0.146933333333 rpy=0 0 0, axis 0 1 0, limit lower=-1.57 upper=1.57 effort=50 velocity=40
- added joint body_tail_joint_5: type revolute, parent tail_link_4, child tail_link_5, origin xyz=0 0 0.146933333333 rpy=0 0 0, axis 0 1 0, limit lower=-1.57 upper=1.57 effort=50 velocity=40
- joint body_tail_joint_0: axis 1 0 0 -> 0 1 0
- joint tail_link_mass_joint: origin xyz=0 0 0.8816 -> xyz=0 0 0.146933333333; parent tail_link_0 -> tail_link_5

File: quad_simulator/spirit_description/xacro/spirit_gazebo_tail.urdf.xacro (robot description, xacro)
@@ -64,5 +64,7 @@
 	<xacro:property name="jointSpeedLimit" value="37.7" /> <!-- Original: 30 -->
 	<xacro:property name="jointEffortLimit" value="21" /> <!-- Original: 40 -->
-	<xacro:property name="tailLength" value="${0.8816/2}" />
+	<xacro:property name="tailNum" value="2" />
+	<xacro:property name="tailLength" value="${0.8816/tailNum}" />
+	<xacro:property name="tailLinkMass" value="${1e-03}" />
 	<!-- Plugins -->
 	<gazebo>
@@ -404,4 +406,5 @@
 	</gazebo>
 	<!-- TAIL -->
+	<!-- Remark: Need to incorporate reasonable mass & inertia calc wrt tailLength -->
 	<!-- Tail Links -->
 	<link name="tail_link_0">
@@ -414,6 +417,9 @@
 		</visual>
 		<inertial>
-			<mass value="1e-03" />
-			<inertia ixx="1e-04" ixy="0" ixz="0" iyy="1e-04" iyz="0.0" izz="1e-04" />
+			<origin xyz="0 0 ${tailLength/2}" rpy="0 0 0" />
+			<mass value="${tailLinkMass}" />
+			<!--<inertia ixx="${tailLinkMass/12*(3*0.02*0.02 + tailLength*tailLength)}" ixy="0" ixz="0" iyy="${tailLinkMass/12*(3*0.02*0.02 + tailLength*tailLength)}" iyz="0.0" izz="${tailLinkMass*(0.02*0.02)/2}" /> -->
+			<!-- Assume inertia of a sphere & scale base of 2/5MR^2 -->
+			<inertia ixx="${1e-04/(tailNum*tailNum)}" ixy="0" ixz="0" iyy="${1e-04/(tailNum*tailNum)}" iyz="0" izz="${1e-04/(tailNum*tailNum)}" />
 		</inertial>
 		<!-- No need to add collision boxes for this -->
@@ -431,8 +437,8 @@
 		</visual>
 		<inertial>
-			<mass value="1e-03" />
-			<inertia ixx="1e-04" ixy="0" ixz="0" iyy="1e-04" iyz="0.0" izz="1e-04" />
+			<origin xyz="0 0 ${tailLength/2}" rpy="0 0 0" />
+			<mass value="${tailLinkMass}" />
+			<inertia ixx="${1e-04/(tailNum*tailNum)}" ixy="0" ixz="0" iyy="${1e-04/(tailNum*tailNum)}" iyz="0" izz="${1e-04/(tailNum*tailNum)}" />
 		</inertial>
-		<!-- No need to add collision boxes for this -->
 	</link>
 	<gazebo reference="tail_link_1">
@@ -456,4 +462,5 @@
 	</gazebo>
 	<!-- Tail Joints -->
+	<!-- Non-planar Tail -->
 	<joint name="body_tail_joint_0" type="revolute">
 		<parent link="body" />
@@ -461,5 +468,5 @@
 		<axis xyz="1 0 0" />
 		<origin xyz="0 0 0" rpy="0 0 0" />
-		<limit effort="50" lower="-1.57" upper="1.57" velocity="1000000" />
+		<limit effort="50" lower="-1.57" upper="1.57" velocity="40" />
 		<dynamics damping="0.0" friction="0.0" />
 	</joint>
@@ -469,5 +476,5 @@
 		<axis xyz="0 1 0" />
 		<origin xyz="0 0 ${tailLength}" rpy="0 0 0" />
-		<limit effort="50" lower="-1.57" upper="1.57" velocity="1000000" />
+		<limit effort="50" lower="-1.57" upper="1.57" velocity="40" />
 		<dynamics damping="0.0" friction="0.0" />
 	</joint>
